File: pcb/artboard.sch (KiCad schematic (older format))
At the start: 25 parts, among them J2 OLED, SW1 SW_PUSH, SW2 SW_PUSH, SW22 SW_SPDT, SW23 SW_SPDT, SW3 SW_PUSH, SW4 SW_PUSH, SW5 SW_PUSH, SW6 SW_PUSH, SW7 SW_PUSH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

Commit message: fix symbol library
Parts:
- RSW1, RSW2, SW1, SW2, SW3, SW4, SW5, SW6, SW7, SW8: symbol kbd:SW_PUSH -> artboard-rescue:SW_PUSH-kbd
- U1: symbol kbd:ProMicro -> artboard:ProMicro
Changed lines of the file:
@@
 $EndDescr
 $Comp
-L kbd:SW_PUSH RSW1
+L artboard-rescue:SW_PUSH-kbd RSW1
 U 1 1 5A5EB9E2
 P 1420 2085
@@
 	1200 2835 1650 2835
 $Comp
-L kbd:SW_PUSH SW7
+L artboard-rescue:SW_PUSH-kbd SW7
 U 1 1 5A5E2D6E
 P 2390 1490
@@
 $EndComp
 $Comp
-L kbd:SW_PUSH SW8
+L artboard-rescue:SW_PUSH-kbd SW8
 U 1 1 5A5E2D26
 P 3090 1490
@@
 $EndComp
 $Comp
-L kbd:SW_PUSH SW1
+L artboard-rescue:SW_PUSH-kbd SW1
 U 1 1 5A5E2B19
 P 990 1100
@@
 $EndComp
 $Comp
-L kbd:SW_PUSH SW4
+L artboard-rescue:SW_PUSH-kbd SW4
 U 1 1 5A5E2908
 P 3090 1100
@@
 $EndComp
 $Comp
-L kbd:SW_PUSH SW3
+L artboard-rescue:SW_PUSH-kbd SW3
 U 1 1 5A5E27F9
 P 2390 1100
@@
 raw
 $Comp
-L kbd:ProMicro U1
+L artboard:ProMicro U1
 U 1 1 5A5E14C2
 P 5065 2865
@@
 $EndComp
 $Comp
-L kbd:SW_PUSH SW6
+L artboard-rescue:SW_PUSH-kbd SW6
 U 1 1 5A5E295E
 P 1690 1490
@@
 $EndComp
 $Comp
-L kbd:SW_PUSH SW5
+L artboard-rescue:SW_PUSH-kbd SW5
 U 1 1 5A5E2933
 P 990 1490
@@
 $EndComp
 $Comp
-L kbd:SW_PUSH SW2
+L artboard-rescue:SW_PUSH-kbd SW2
 U 1 1 5A5E2699
 P 1690 1100
@@
 $EndComp
 $Comp
-L kbd:SW_PUSH RSW2
+L artboard-rescue:SW_PUSH-kbd RSW2
 U 1 1 607A3E8D
 P 1405 2385

Commit message: fix some rescued symbols
Parts:
- SW1, SW2, SW3, SW4, SW5, SW6, SW7, SW8: symbol artboard-rescue:SW_PUSH-kbd -> artboard:SW_PUSH
Changed lines of the file:
@@
 	1200 2835 1650 2835
 $Comp
-L artboard-rescue:SW_PUSH-kbd SW7
+L artboard:SW_PUSH SW7
 U 1 1 5A5E2D6E
 P 2390 1490
@@
 $EndComp
 $Comp
-L artboard-rescue:SW_PUSH-kbd SW8
+L artboard:SW_PUSH SW8
 U 1 1 5A5E2D26
 P 3090 1490
@@
 $EndComp
 $Comp
-L artboard-rescue:SW_PUSH-kbd SW1
+L artboard:SW_PUSH SW1
 U 1 1 5A5E2B19
 P 990 1100
@@
 $EndComp
 $Comp
-L artboard-rescue:SW_PUSH-kbd SW4
+L artboard:SW_PUSH SW4
 U 1 1 5A5E2908
 P 3090 1100
@@
 $EndComp
 $Comp
-L artboard-rescue:SW_PUSH-kbd SW3
+L artboard:SW_PUSH SW3
 U 1 1 5A5E27F9
 P 2390 1100
@@
 $EndComp
 $Comp
-L artboard-rescue:SW_PUSH-kbd SW6
+L artboard:SW_PUSH SW6
 U 1 1 5A5E295E
 P 1690 1490
@@
 $EndComp
 $Comp
-L artboard-rescue:SW_PUSH-kbd SW5
+L artboard:SW_PUSH SW5
 U 1 1 5A5E2933
 P 990 1490
@@
 $EndComp
 $Comp
-L artboard-rescue:SW_PUSH-kbd SW2
+L artboard:SW_PUSH SW2
 U 1 1 5A5E2699
 P 1690 1100
